Commit message: Initial Controller Configurations

File: src/palm_trimmer_description/urdf/palm_trimmer.urdf.xacro (robot description, xacro)
@@ -61,3 +61,28 @@
     <limit lower="0.0" upper="0.50" effort="100" velocity="0.20"/>
   </joint>
+  <ros2_control name="GazeboSimSystem" type="system">
+    <hardware>
+      <plugin>gz_ros2_control/GazeboSimSystem</plugin>
+    </hardware>
+    <joint name="arm_extension_joint">
+      <command_interface name="position">
+        <param name="min">0.0</param>
+        <param name="max">0.50</param>
+      </command_interface>
+      <state_interface name="position">
+        <param name="initial_value">0.0</param>
+      </state_interface>
+      <state_interface name="velocity"/>
+      <state_interface name="effort"/>
+    </joint>
+  </ros2_control>
+  <gazebo>
+    <plugin
+      filename="gz_ros2_control-system"
+      name="gz_ros2_control::GazeboSimROS2ControlPlugin">
+      <parameters>
+        $(find palm_trimmer_description)/config/controllers.yaml
+      </parameters>
+    </plugin>
+  </gazebo>
 </robot>
